Commit message: fix

File: pybullet_robot_envs/robot_data/franka_description/cube_small.urdf (robot description, URDF)
Before this commit: robot cube.urdf, 1 links, 0 joints
Links:
- link baseLink: mass .1 -> .2; geometry collision box size=.1 .1 .1; visual mesh filename=cube.obj scale=.1 .1 .1

File: pybullet_robot_envs/robot_data/franka_description/robots/panda_arm_physics.urdf (robot description, URDF)
Before this commit: robot panda, 12 links, 11 joints
Joints:
- joint panda_joint1: limit lower=-2.8973 upper=2.8973 effort=87 velocity=2.1750 -> lower=-1 upper=1 effort=87 velocity=2.1750
- joint panda_joint2: limit lower=-1.7628 upper=1.7628 effort=87 velocity=2.1750 -> lower=0 upper=1.7628 effort=87 velocity=2.1750; origin xyz=0 0 0 rpy=-1.57079632679 0 0 -> xyz=0 0 0 rpy=-1.57079632679 1.5 0
