Commit message: update figure of robot envs

File: pybullet_robot_envs/robot_data/franka_panda/panda_model.urdf (robot description, URDF)
Before this commit: robot panda, 22 links, 21 joints
Links:
- removed link camera_color_frame
- removed link camera_color_optical_frame
- removed link camera_depth_frame
- removed link camera_depth_optical_frame
- removed link camera_left_ir_frame
- removed link camera_left_ir_optical_frame
- removed link camera_link
- removed link camera_right_ir_frame
- removed link camera_right_ir_optical_frame
Joints:
- removed joint camera_color_joint
- removed joint camera_color_optical_joint
- removed joint camera_depth_joint
- removed joint camera_depth_optical_joint
- removed joint camera_joint
- removed joint camera_left_ir_joint
- removed joint camera_left_ir_optical_joint
- removed joint camera_right_ir_joint
- removed joint camera_right_ir_optical_joint
